File: atl100_tht/atl100_modules.kicad_sch (KiCad schematic)
At the start: 7 parts

Commit message: feat: Version 1.0.0
Parts:
- removed D1: LED_RKGB, symbol Device:LED_RKGB
- removed R11: 67R, symbol Device:R
- removed R12: 42R, symbol Device:R
- removed R13: 17R, symbol Device:R
- removed U3: ~, symbol AgroTechLab:RS485_to_TTL_Module
- removed U4: ~, symbol AgroTechLab:HD-38_Module
- added U3: ~, AgroTechLab:HW-519, symbol AgroTechLab:RS-485 to TTL Module
- U5: value ~ -> ADC 4~20mA; footprint (none) -> AgroTechLab:ADC_4_20_mA_Module; Manufacturer (none) -> Circuitar; Part Number (none) -> ADC 4~20mA
Connections:
- net +3V3: now also U3.1 (VCC)
- net GND: now also U3.4 (GND)
- net MCU_RXD - RS485_TXD: now also U3.2 (TXD)
- net MCU_TXD - RS485_RXD: now also U3.3 (RXD)
- new net RS485_A+: U3.5 (A+)
- new net RS485_B-: U3.6 (B-)
- new net RS485_COM: U3.7 (COM)
- no-connect marks 25 -> 24
Other:
- note removed: "HD-38"
- note removed: "HD-38 (Soil Moisture)"
- note removed: "RGB LED (Cathode)"
- note removed: "Soil Moisture: 0% ~ 100%"
