File: atl100_tht/atl100_terminals.kicad_sch (KiCad schematic)
At the start: 6 parts, among them J1 Screw_Terminal_01x02, J2 Screw_Terminal_01x02, J3 Screw_Terminal_01x02, J4 Screw_Terminal_01x02, J5 Screw_Terminal_01x03, J6 Screw_Terminal_01x02

Commit message: feat: Version 1.0.0
Parts:
- removed J2: Screw_Terminal_01x02, symbol Connector:Screw_Terminal_01x02
- removed J5: Screw_Terminal_01x03, symbol Connector:Screw_Terminal_01x03
- added H1, H2, H3, H4: MountingHole_Pad, MountingHole:MountingHole_2.2mm_M2_Pad_Via, symbol Mechanical:MountingHole_Pad
- added J1: Conn_01x04_Pin, Connector_PinHeader_2.54mm:PinHeader_1x04_P2.54mm_Vertical, symbol Connector:Conn_01x04_Pin
- added J6, J7: Screw_Terminal_01x04, TerminalBlock_Phoenix:TerminalBlock_Phoenix_MKDS-1,5-4-5.08_1x04_P5.08mm_Horizontal, symbol Connector:Screw_Terminal_01x04
- added J8: Screw_Terminal_01x06, TerminalBlock_Phoenix:TerminalBlock_Phoenix_MKDS-1,5-6-5.08_1x06_P5.08mm_Horizontal, symbol Connector:Screw_Terminal_01x06
- added R1: 67R, Resistor_THT:R_Axial_DIN0207_L6.3mm_D2.5mm_P10.16mm_Horizontal, symbol Device:R
- added R2: 42R, Resistor_THT:R_Axial_DIN0207_L6.3mm_D2.5mm_P10.16mm_Horizontal, symbol Device:R
- added R3: 17R, Resistor_THT:R_Axial_DIN0207_L6.3mm_D2.5mm_P10.16mm_Horizontal, symbol Device:R
- J2: renamed from J1; footprint (none) -> TerminalBlock_Phoenix:TerminalBlock_Phoenix_MKDS-1,5-2-5.08_1x02_P5.08mm_Horizontal; Manufacturer CUI Devices -> Std; Part Number TB001-500-02BE -> Std
- J3, J4: footprint (none) -> TerminalBlock_Phoenix:TerminalBlock_Phoenix_MKDS-1,5-2-5.08_1x02_P5.08mm_Horizontal; Manufacturer CUI Devices -> Std; Part Number TB001-500-02BE -> Std
- J5: renamed from J6; footprint (none) -> TerminalBlock_Phoenix:TerminalBlock_Phoenix_MKDS-1,5-2-5.08_1x02_P5.08mm_Horizontal; Manufacturer CUI Devices -> Std; Part Number TB001-500-02BE -> Std
Connections:
- net +3V3: now also J6.1 (Pin_1)
- net +5V: now also J7.1 (Pin_1)
- net GND: now also H1.1, H2.1, H3.1, H4.1, J1.1 (Pin_1), J6.2 (Pin_2), J8.1 (Pin_1)
- net I2C_SCL: now also J6.3 (Pin_3)
- net I2C_SDA: now also J6.4 (Pin_4)
- new net: J1.4 (Pin_4), R3.1
- new net: J1.3 (Pin_3), R2.1
- new net: J1.2 (Pin_2), R1.1
- new net AI1: J8.3 (Pin_3)
- new net AI2: J8.4 (Pin_4)
- new net AI3: J8.5 (Pin_5)
- new net AI4: J8.6 (Pin_6)
- new net LED_BLUE: R3.2
- new net LED_GREEN: R2.2
- new net LED_RED: R1.2
- new net RS485_A+: J7.2 (Pin_2)
- new net RS485_B-: J7.3 (Pin_3)
- new net RS485_COM: J7.4 (Pin_4)
- no-connect marks 0 -> 1
Other:
- note added: "Analog Inputs"
- note added: "RGB LED (Cathode)"
- note added: "RS-485"
- note removed: "DS18B20"
- moved on the sheet: J2, J3, J4, J5
