File: atl100_tht/atl100_tht.kicad_sch (KiCad schematic)
At the start: 0 parts

Commit message: feat: Schematic updated (v0.1.0)
Other:
- removed sheet Analog Inputs
- removed sheet Digital Inputs
- removed sheet RS-485
- removed sheet mPCIe
- added sheet MCU (atl100_mcu.kicad_sch)
- added sheet Modules (atl100_modules.kicad_sch)
- sheet Power Supply: file power_supply.kicad_sch -> atl100_power_supply.kicad_sch
- sheet Terminals: file terminals.kicad_sch -> atl100_terminals.kicad_sch
- note added: "ATL-100 (Multiparametric Station)"
- note added: "Components Format: THT Internal Modules: - MCU (ESP32-S3) - XL4005 (Voltage Regulator - Step Down) - Voltage Sensor (power supply voltage) - HD-38 (soil moisture) - HW-519 (RS-485) - RGB LED External Modules: - BME-280 (air temperature, air humidity, atmospherical pressure) - Pluviometer (rain amount) - Anemometer (wind speed) - Windsock (wind direction) - ADC 4mA - 20mA (4x ports)"
- title: ATL100 (Multiparametric Station) -> ATL100 (Multiparametric Station) - THT Based
Changed lines of the file:
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@@
 	(paper "A4")
 	(title_block
-		(title "ATL100 (Multiparametric Station)")
-		(date "2024-07-01")
+		(title "ATL100 (Multiparametric Station) - THT Based")
+		(date "2024-09-06")
 		(rev "v0.1.0-alpha")
 		(company "AgroTechLab (Laboratório de Desenvolvimento de Tecnologias para o Agrongócio)")
@@
 		(comment 4 "Total Supply Current: ??mA (??mA)")
 	)
+	(rectangle
+		(start 31.115 34.29)
+		(end 106.68 72.39)
+		(stroke
+			(width 0)
+			(type dash)
+			(color 9 23 255 1)
+		)
+		(fill
+			(type none)
+		)
+	)
+	(text "Components Format: THT\n\nInternal Modules:\n   - MCU (ESP32-S3)\n   - XL4005 (Voltage Regulator - Step Down)\n   - Voltage Sensor (power supply voltage)\n   - HD-38 (soil moisture)\n   - HW-519 (RS-485)\n   - RGB LED\n\nExternal Modules:\n   - BME-280 (air temperature, air humidity, atmospherical pressure)\n   - Pluviometer (rain amount)\n   - Anemometer (wind speed)\n   - Windsock (wind direction)\n   - ADC 4mA - 20mA (4x ports)"
+		(exclude_from_sim no)
+		(at 32.512 70.358 0)
+		(effects
+			(font
+				(size 1.27 1.27)
+				(color 9 23 255 1)
+			)
+			(justify left bottom)
+		)
+	)
+	(text "ATL-100 (Multiparametric Station)"
+		(exclude_from_sim no)
+		(at 31.75 36.957 0)
+		(effects
+			(font
+				(size 1.27 1.27)
+				(thickness 0.254)
+				(bold yes)
+				(color 9 23 255 1)
+			)
+			(justify left bottom)
+		)
+	)
 	(sheet
-		(at 218.44 138.43)
+		(at 197.485 153.67)
 		(size 12.7 7.62)
 		(fields_autoplaced yes)
@@
 			(color 0 0 0 0.0000)
 		)
-		(property "Sheetname" "Analog Inputs"
-			(at 218.44 137.7184 0)
+		(property "Sheetname" "Modules"
+			(at 197.485 152.9584 0)
 			(effects
 				(font
@@
 			)
 		)
-		(property "Sheetfile" "analog_inputs.kicad_sch"
-			(at 218.44 146.6346 0)
+		(property "Sheetfile" "atl100_modules.kicad_sch"
+			(at 197.485 161.8746 0)
 			(effects
 				(font
@@
 				)
 				(justify left top)
+				(hide yes)
 			)
 		)
 		(instances
-			(project "atl100"
+			(project "atl100_tht"
 				(path "/9f25808e-b525-4dd9-b9a0-a085d29b6aa9"
-					(page "4")
+					(page "5")
 				)
 			)
@@
 	)
 	(sheet
-		(at 218.44 153.67)
+		(at 197.3673 139.0856)
 		(size 12.7 7.62)
 		(fields_autoplaced yes)
@@
 			(color 0 0 0 0.0000)
 		)
-		(property "Sheetname" "Digital Inputs"
-			(at 218.44 152.9584 0)
+		(property "Sheetname" "MCU"
+			(at 197.3673 138.374 0)
 			(effects
 				(font
@@
 			)
 		)
-		(property "Sheetfile" "digital_inputs.kicad_sch"
-			(at 218.44 161.8746 0)
+		(property "Sheetfile" "atl100_mcu.kicad_sch"
+			(at 197.3673 147.2902 0)
 			(effects
 				(font
@@
 				)
 				(justify left top)
+				(hide yes)
 			)
 		)
 		(instances
-			(project "atl100"
+			(project "atl100_tht"
 				(path "/9f25808e-b525-4dd9-b9a0-a085d29b6aa9"
-					(page "3")
+					(page "4")
 				)
 			)
@@
 	)
 	(sheet
-		(at 179.07 138.43)
-		(size 12.7 7.62)
-		(fields_autoplaced yes)
-		(stroke
-			(width 0.1524)
-			(type solid)
-		)
-		(fill
-			(color 0 0 0 0.0000)
-		)
-		(property "Sheetname" "RS-485"
-			(at 179.07 137.7184 0)
-			(effects
-				(font
-					(size 1.27 1.27)
-				)
-				(justify left bottom)
-			)
-		)
-		(property "Sheetfile" "rs485.kicad_sch"
-			(at 179.07 146.6346 0)
-			(effects
-				(font
-					(size 1.27 1.27)
-				)
-				(justify left top)
-			)
-		)
-		(instances
-			(project "atl100"
-				(path "/9f25808e-b525-4dd9-b9a0-a085d29b6aa9"
-					(page "5")
-				)
-			)
-		)
-	)
-	(sheet
-		(at 179.07 153.67)
+		(at 177.8 139.065)
 		(size 12.7 7.62)
 		(fields_autoplaced yes)
@@
 		)
 		(property "Sheetname" "Power Supply"
-			(at 179.07 152.9584 0)
+			(at 177.8 138.3534 0)
 			(effects
 				(font
@@
 			)
 		)
-		(property "Sheetfile" "power_supply.kicad_sch"
-			(at 179.07 161.8746 0)
+		(property "Sheetfile" "atl100_power_supply.kicad_sch"
+			(at 177.8 147.2696 0)
 			(effects
 				(font
@@
 				)
 				(justify left top)
+				(hide yes)
 			)
 		)
 		(instances
-			(project "atl100"
+			(project "atl100_tht"
 				(path "/9f25808e-b525-4dd9-b9a0-a085d29b6aa9"
-					(page "2")
+					(page "3")
 				)
 			)
@@
 	)
 	(sheet
-		(at 256.54 153.67)
-		(size 12.7 7.62)
-		(fields_autoplaced yes)
-		(stroke
-			(width 0.1524)
-			(type solid)
-		)
-		(fill
-			(color 0 0 0 0.0000)
-		)
-		(property "Sheetname" "mPCIe"
-			(at 256.54 152.9584 0)
-			(effects
-				(font
-					(size 1.27 1.27)
-				)
-				(justify left bottom)
-			)
-		)
-		(property "Sheetfile" "mpcie.kicad_sch"
-			(at 256.54 161.8746 0)
-			(effects
-				(font
-					(size 1.27 1.27)
-				)
-				(justify left top)
-			)
-		)
-		(instances
-			(project "atl100"
-				(path "/9f25808e-b525-4dd9-b9a0-a085d29b6aa9"
-					(page "6")
-				)
-			)
-		)
-	)
-	(sheet
-		(at 256.54 139.7)
+		(at 177.8 153.67)
 		(size 12.7 7.62)
 		(fields_autoplaced yes)
@@
 		)
 		(property "Sheetname" "Terminals"
-			(at 256.54 138.9884 0)
+			(at 177.8 152.9584 0)
 			(effects
 				(font
@@
 			)
 		)
-		(property "Sheetfile" "terminals.kicad_sch"
-			(at 256.54 147.9046 0)
+		(property "Sheetfile" "atl100_terminals.kicad_sch"
+			(at 177.8 161.8746 0)
 			(effects
 				(font
@@
 				)
 				(justify left top)
+				(hide yes)
 			)
 		)
 		(instances
-			(project "atl100"
+			(project "atl100_tht"
 				(path "/9f25808e-b525-4dd9-b9a0-a085d29b6aa9"
-					(page "7")
+					(page "2")
 				)
 			)

Commit message: feat: Version 1.0.0
Other:
- sheet Modules renamed RS-485
- added sheet Analog Inputs (atl100_ai.kicad_sch)
- added sheet LTE (atl100_lte.kicad_sch)
- sheet RS-485: file atl100_modules.kicad_sch -> atl100_rs485.kicad_sch
- note added: "Air Temperature: -40ºC ~ 85ºC (0,01ºC / ±1ºC) Air Humidity: 0% ~ 100% (0,008% / ±3%) Atmospheric Pressure: 300hPa ~ 1100hPa (0,18hPa / ±1hPa) I2C Addr: 0x76 (SDO Low) 0x77 (SDO High)"
- note added: "BME280"
- note added: "Components Format: THT Internal Modules: - MCU (ESP32-S3) - XL4005 (Voltage Regulator - Step Down) - Voltage Sensor (power supply voltage) - HW-519 (RS-485) - RGB LED External Modules: - BME-280 (I2C port) - Air Temperature (ºC) - Air Humidity (%) - Atmospherical Pressure (mmHg) - Pluviometer (pulse port) - Rain Amount (mm) - Anemometer (pulse port) - Wind Speed (m/sec. or Km/h) - Windsock (ADC p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"
- note added: "DS18B20"
- note added: "Soil Temperature: -55ºC ~ 125ºC (0,01ºC / ±0,5ºC) Resolution: 9 ~ 12 (adjustable)"
- note removed: "Components Format: THT Internal Modules: - MCU (ESP32-S3) - XL4005 (Voltage Regulator - Step Down) - Voltage Sensor (power supply voltage) - HD-38 (soil moisture) - HW-519 (RS-485) - RGB LED External Modules: - BME-280 (air temperature, air humidity, atmospherical pressure) - Pluviometer (rain amount) - Anemometer (wind speed) - Windsock (wind direction) - ADC 4mA - 20mA (4x ports)"
Changed lines of the file:
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@@
 	(title_block
 		(title "ATL100 (Multiparametric Station) - THT Based")
-		(date "2024-09-06")
-		(rev "v0.1.0-alpha")
+		(date "2024-10-27")
+		(rev "v1.0.0")
 		(company "AgroTechLab (Laboratório de Desenvolvimento de Tecnologias para o Agrongócio)")
 		(comment 1 "IFSC/Lages (Instituto Federal de Santa Catarina)")
@@
 	)
 	(rectangle
-		(start 31.115 34.29)
-		(end 106.68 72.39)
+		(start 116.8512 68.4903)
+		(end 180.3512 76.581)
 		(stroke
 			(width 0)
@@
 		)
 	)
-	(text "Components Format: THT\n\nInternal Modules:\n   - MCU (ESP32-S3)\n   - XL4005 (Voltage Regulator - Step Down)\n   - Voltage Sensor (power supply voltage)\n   - HD-38 (soil moisture)\n   - HW-519 (RS-485)\n   - RGB LED\n\nExternal Modules:\n   - BME-280 (air temperature, air humidity, atmospherical pressure)\n   - Pluviometer (rain amount)\n   - Anemometer (wind speed)\n   - Windsock (wind direction)\n   - ADC 4mA - 20mA (4x ports)"
-		(exclude_from_sim no)
-		(at 32.512 70.358 0)
-		(effects
-			(font
-				(size 1.27 1.27)
-				(color 9 23 255 1)
-			)
-			(justify left bottom)
-		)
-	)
-	(text "ATL-100 (Multiparametric Station)"
-		(exclude_from_sim no)
-		(at 31.75 36.957 0)
+	(rectangle
+		(start 116.84 53.34)
+		(end 180.34 67.31)
+		(stroke
+			(width 0)
+			(type dash)
+			(color 9 23 255 1)
+		)
+		(fill
+			(type none)
+		)
+	)
+	(rectangle
+		(start 31.115 34.29)
+		(end 106.68 106.045)
+		(stroke
+			(width 0)
+			(type dash)
+			(color 9 23 255 1)
+		)
+		(fill
+			(type none)
+		)
+	)
+	(text "Soil Temperature: -55ºC ~ 125ºC (0,01ºC / ±0,5ºC)\nResolution: 9 ~ 12 (adjustable)"
+		(exclude_from_sim no)
+		(at 117.475 75.565 0)
+		(effects
+			(font
+				(size 1.27 1.27)
+				(color 9 23 255 1)
+			)
+			(justify left bottom)
+		)
+	)
+	(text "DS18B20"
+		(exclude_from_sim no)
+		(at 117.4862 71.1573 0)
 		(effects
 			(font
@@
 			)
 			(justify left bottom)
+		)
+	)
+	(text "BME280"
+		(exclude_from_sim no)
+		(at 117.475 56.007 0)
+		(effects
+			(font
+				(size 1.27 1.27)
+				(thickness 0.254)
+				(bold yes)
+				(color 9 23 255 1)
+			)
+			(justify left bottom)
+		)
+	)
+	(text "Air Temperature: -40ºC ~ 85ºC (0,01ºC / ±1ºC)\nAir Humidity: 0% ~ 100% (0,008% / ±3%)\nAtmospheric Pressure: 300hPa ~ 1100hPa (0,18hPa / ±1hPa)\nI2C Addr: 0x76 (SDO Low)\n          0x77 (SDO High)"
+		(exclude_from_sim no)
+		(at 117.729 66.421 0)
+		(effects
+			(font
+				(size 1.27 1.27)
+				(color 9 23 255 1)
+			)
+			(justify left bottom)
+		)
+	)
+	(text "Components Format: THT\n\nInternal Modules:\n   - MCU (ESP32-S3)\n   - XL4005 (Voltage Regulator - Step Down)\n   - Voltage Sensor (power supply voltage)\n   - HW-519 (RS-485)\n   - RGB LED\n\nExternal Modules:\n   - BME-280 (I2C port)\n      - Air Temperature (ºC)\n      - Air Humidity (%)\n      - Atmospherical Pressure (mmHg)\n   - Pluviometer (pulse port)\n      - Rain Amount (mm)\n   - Anemometer (pulse port)\n      - Wind Speed (m/sec. or Km/h)\n   - Windsock (ADC port)\n      - Wind Direction (N, NE, E, SE, S, SW, W, NW)\n   - ADC 4mA - 20mA (4x ports)\n   - Soil Sensor (RS-485 port)\n      - Temperature (%)\n      - Moisture (ºC)\n      - PH (index)\n      - Conductivity (µs/cm)\n      - Nitrogen (mg/Kg)\n      - Potassium (mg/Kg)\n      - Calcium (mg/Kg)"
+		(exclude_from_sim no)
+		(at 33.782 97.282 0)
+		(effects
+			(font
+				(size 1.27 1.27)
+				(color 9 23 255 1)
+			)
+			(justify left bottom)
+		)
+	)
+	(text "ATL-100 (Multiparametric Station)"
+		(exclude_from_sim no)
+		(at 31.75 36.957 0)
+		(effects
+			(font
+				(size 1.27 1.27)
+				(thickness 0.254)
+				(bold yes)
+				(color 9 23 255 1)
+			)
+			(justify left bottom)
+		)
+	)
+	(sheet
+		(at 215.9 153.67)
+		(size 12.7 7.62)
+		(fields_autoplaced yes)
+		(stroke
+			(width 0.1524)
+			(type solid)
+		)
+		(fill
+			(color 0 0 0 0.0000)
+		)
+		(property "Sheetname" "LTE"
+			(at 215.9 152.9584 0)
+			(effects
+				(font
+					(size 1.27 1.27)
+				)
+				(justify left bottom)
+			)
+		)
+		(property "Sheetfile" "atl100_lte.kicad_sch"
+			(at 215.9 161.8746 0)
+			(effects
+				(font
+					(size 1.27 1.27)
+				)
+				(justify left top)
+				(hide yes)
+			)
+		)
+		(instances
+			(project "atl100_tht"
+				(path "/9f25808e-b525-4dd9-b9a0-a085d29b6aa9"
+					(page "7")
+				)
+			)
+		)
+	)
+	(sheet
+		(at 215.265 139.065)
+		(size 12.7 7.62)
+		(fields_autoplaced yes)
+		(stroke
+			(width 0.1524)
+			(type solid)
+		)
+		(fill
+			(color 0 0 0 0.0000)
+		)
+		(property "Sheetname" "Analog Inputs"
+			(at 215.265 138.3534 0)
+			(effects
+				(font
+					(size 1.27 1.27)
+				)
+				(justify left bottom)
+			)
+		)
+		(property "Sheetfile" "atl100_ai.kicad_sch"
+			(at 215.265 147.2696 0)
+			(effects
+				(font
+					(size 1.27 1.27)
+				)
+				(justify left top)
+				(hide yes)
+			)
+		)
+		(instances
+			(project "atl100_tht"
+				(path "/9f25808e-b525-4dd9-b9a0-a085d29b6aa9"
+					(page "6")
+				)
+			)
 		)
 	)
@@
 			(color 0 0 0 0.0000)
 		)
-		(property "Sheetname" "Modules"
+		(property "Sheetname" "RS-485"
 			(at 197.485 152.9584 0)
 			(effects
@@
 			)
 		)
-		(property "Sheetfile" "atl100_modules.kicad_sch"
+		(property "Sheetfile" "atl100_rs485.kicad_sch"
 			(at 197.485 161.8746 0)
 			(effects
