File: atl100_ai.kicad_sch (KiCad schematic)
At the start: 17 parts, among them U4 ADS1115 Module

Commit message: feat: Main board schematic updated
Other:
- title: ATL-100 (Multiparametric Station) -> ATL-100 (Multiparametric Station) - Main Board
Changed lines of the file:
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@@
 	(paper "A4")
 	(title_block
-		(title "ATL-100 (Multiparametric Station)")
+		(title "ATL-100 (Multiparametric Station) - Main Board")
 		(date "2025-06-01")
 		(rev "v0.2.0")
