File: atl100_mcu.kicad_sch (KiCad schematic)
At the start: 4 parts, among them U2 ESP32-S3

Commit message: feat: Main board schematic updated
Parts:
- added U7: Logical Level Converter, AgroTechLab:Logical Level Converter, symbol AgroTechLab:Logical Level Converter
- renumbered R6 to R3, R7 to R4, R9 to R5, U2 to U4
Connections:
- net +3V3: now also U7.3 (3V3)
- net +5V: now also U7.9 (5V)
- net GND: now also U7.10 (GND), U7.4 (GND)
- net LTE_PEN: now reaches U4.12 (GPIO8/RTC_GPIO8/ADC1_CH7/SUBSPICS1)
- net ADC_ALERT: no longer names the net of U4.30 (MTDO/GPIO40)
- net I2C_SCL renamed I2C_SCL_3V3
- net I2C_SCL_3V3: now also U7.6 (LV4)
- net I2C_SDA renamed I2C_SDA_3V3
- net I2C_SDA_3V3: now also U7.5 (LV3)
- net MCU_RXD - LTE_TXD renamed LTE_TX
- net MCU_RXD - RS485_TXD renamed MCU_RXD0_3V3
- net MCU_RXD0_3V3: now also U7.2 (LV2)
- net MCU_TXD - LTE_RXD renamed LTE_RX
- net MCU_TXD - RS485_RXD renamed MCU_TXD0_3V3
- net MCU_TXD0_3V3: now also U7.1 (LV1)
- new net I2C_SCL_5V: U7.12 (HV4)
- new net I2C_SDA_5V: U7.11 (HV3)
- new net RS485_RX: U7.7 (HV1)
- new net RS485_TX: U7.8 (HV2)
Other:
- title: ATL-100 (Multiparametric Station) -> ATL-100 (Multiparametric Station) - Main Board

Commit message: feat: Updated to v0.2.0
Connections:
- net AN-: now also U4.5 (GPIO5/RTC_GPIO5/ADC1_CH4); no longer U4.35 (SUBSPID/FSPID/SPIIO6/GPIO35)
- net I2C_SCL_3V3: now also U4.20 (GPIO14/RTC_GPIO14/ADC2_CH3/FSPIWP/FSPIDQS/SUBSPIWP); no longer U4.29 (MTDI/GPIO41)
- net I2C_SDA_3V3: now also U4.19 (GPIO13/RTC_GPIO13/ADC2_CH2/FSPIQ/FSPIIO7/SUBSPIQ); no longer U4.28 (MTMS/GPIO42)
- net LED_BLUE: now also U4.39 (SUBSPICLK_P_DIFF/SPICLK_P/GPIO47); no longer U4.6 (GPIO6/RTC_GPIO6/ADC1_CH5)
- net LED_GREEN: now also U4.38 (SUBSPICLK_N_DIFF/SPICLK_N/GPIO48); no longer U4.8 (GPIO15/RTC_GPIO15/ADC2_CH4/U0RTS)
- net LED_RED: now also U4.37 (GPIO45); no longer U4.7 (GPIO7/RTC_GPIO7/ADC1_CH6)
- net LTE_PEN: now also U4.33 (SUBSPIQ/FSPIQ/SPIDQS/GPIO37); no longer U4.12 (GPIO8/RTC_GPIO8/ADC1_CH7/SUBSPICS1)
- net LTE_RX: now also U4.34 (SUBSPICLK/FSPICLK/SPIIO7/GPIO36); no longer U4.10 (GPIO17/RTC_GPIO17/ADC2_CH6/U1TXD)
- net LTE_TX: now also U4.35 (SUBSPID/FSPID/SPIIO6/GPIO35); no longer U4.11 (GPIO18/RTC_GPIO18/ADC2_CH7/U1RXD)
- net MCU_RXD0_3V3: now also U4.16 (GPIO10/RTC_GPIO10/ADC1_CH9/FSPICS0/FSPIIO4/SUBSPICS0); no longer U4.27 (ADC1_CH1/RTC_GPIO2/GPIO2)
- net MCU_TXD0_3V3: now also U4.15 (GPIO9/RTC_GPIO9/ADC1_CH8/FSPIHD/SUBSPIHD); no longer U4.26 (ADC1_CH0/RTC_GPIO1/GPIO1)
- net PL-: now also U4.6 (GPIO6/RTC_GPIO6/ADC1_CH5); no longer U4.31 (SUBSPICS1/MTCK/GPIO39)
- net PWR_SENSOR: now also U4.41 (USB_D+/U1CTS/ADC2_CH9/RTC_GPIO20/GPIO20); no longer U4.20 (GPIO14/RTC_GPIO14/ADC2_CH3/FSPIWP/FSPIDQS/SUBSPIWP)
- net RS485_RX: now also U7.8 (HV2); no longer U7.7 (HV1)
- net RS485_TX: now also U7.7 (HV1); no longer U7.8 (HV2)
- net WS-: now also U4.4 (GPIO4/RTC_GPIO4/ADC1_CH3); no longer U4.40 (RTC_GPIO21/GPIO21)
- net LORA_TX: now reaches U4.30 (MTDO/GPIO40)
- new net LORA_BOOT0: U4.28 (MTMS/GPIO42)
- new net LORA_RST: U4.29 (MTDI/GPIO41)
- new net LORA_RX: U4.31 (SUBSPICS1/MTCK/GPIO39)
- no-connect marks 23 -> 19
Other:
- moved on the sheet: R3, R4, R5
